Commit message: pregrasp+no collision spheres on gripper

File: curobo/curobo/content/assets/robot/franka_description/dual_franka_panda.urdf (robot description, URDF)
Before this commit: robot dual_panda, 32 links, 31 joints
Joints:
- joint base_joint: origin xyz=0.0 -0.45 0.0 rpy=0 0 0 -> xyz=0.0 -0.6 0.0 rpy=0 0 0
- joint base_joint_1: origin xyz=0.0 0.45 0.0 rpy=0 0 0 -> xyz=0.0 0.6 0.0 rpy=0 0 0
