Commit message: dual facing

File: content/assets/robot/franka_description/dual_franka_panda_facing.urdf (robot description, URDF)
Before this commit: robot dual_panda, 32 links, 31 joints
Joints:
- joint base_joint: origin xyz=0.0 -0.6 0.0 rpy=0 0 0 -> xyz=0.0 -0.7 0.0 rpy=0 0 0
- joint base_joint_1: origin xyz=0.0 0.6 0.0 rpy=0 0 0 -> xyz=0.0 0.7 0.0 rpy=0 0 0
- joint panda_fixed: origin xyz=0 0 0.0 rpy=0 0 0.0 -> xyz=0 0 0.0 rpy=0 0 2
- joint panda_fixed_1: origin xyz=0 0 0.0 rpy=0 0 0.0 -> xyz=0 0 0.0 rpy=0 0 -2
